File: dual-knobbos.kicad_pcb (KiCad board)
At the start: 2 copper layers, 34 parts, among them J1 USB_C_Receptacle_USB2.0, SW1 SW_Push, SW2 Rotary_Encoder_Switch, SW3 Rotary_Encoder_Switch, U1 ATmega32U4-AU, Y1 16MHz

Commit message: mid commit
Parts:
- C1, C2, C3, C4, C5, C6, C7, F1, R1, R2, R3, R4, R5, R6, SW1, U1, Y1: moved to B.Cu
- moved MX1 137.0 mm to (4.76, 61.1)
- moved D1 131.5 mm to (3.17, 66.7)
- moved D5 121.1 mm to (42.1, 66.7)
- moved D2 118.2 mm to (3.17, 86.5)
- moved J1 113.1 mm to (-7.94, 56.4)
- moved D3 99.9 mm to (23.0, 67.5)
- moved D4 93.8 mm to (22.2, 85.7)
- moved MX6 89.3 mm to (42.9, 80.2)
- moved MX4 88.2 mm to (23.8, 80.2)
- moved MX2 87.1 mm to (4.76, 80.2)
- moved MX5 86.1 mm to (42.9, 61.1)
- moved MX3 85.2 mm to (23.8, 61.1)
- moved D7 79.1 mm to (76.2, 53.6)
- moved D6 72.8 mm to (41.9, 85.7)
- moved C4 72.7 mm to (147.4, 69.3), turned to 90 degrees
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
Commit message: some commit idk
Parts:
- moved J1 171.3 mm to (148.7, 125.7), turned to 180 degrees
- moved SW1 145.7 mm to (193.7, 137.3), turned to 270 degrees
- moved MX1 135.6 mm to (115.9, 138.9)
- moved MX2 135.6 mm to (115.9, 158.0)
- moved MX3 135.6 mm to (134.9, 138.9)
- moved MX4 135.6 mm to (134.9, 158.0)
- moved MX5 135.6 mm to (154.0, 138.9)
- moved MX6 135.6 mm to (154.0, 158.0)
- moved D7 133.0 mm to (188.1, 125.4), turned to 270 degrees
- moved D1 132.8 mm to (122.2, 125.4), turned to 270 degrees
- moved D2 128.8 mm to (125.4, 127.0), turned to 270 degrees
- moved D5 128.5 mm to (156.4, 125.4), turned to 270 degrees
- moved D8 120.9 mm to (190.5, 127.0), turned to 270 degrees
- moved D3 120.4 mm to (128.6, 125.4), turned to 270 degrees
- moved D4 117.1 mm to (131.8, 127.0), turned to 270 degrees
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Connections:
- U1 pad 26: Net-(U1-Pad26) -> COL3
- U1 pad 27: Net-(U1-Pad27) -> ENC0A
- U1 pad 28: Net-(U1-Pad28) -> ENC0B
- U1 pad 29: Net-(U1-Pad29) -> ENC1A
- U1 pad 30: Net-(U1-Pad30) -> ENC1B
- U1 pad 38: Net-(U1-Pad38) -> COL3
- U1 pad 39: Net-(U1-Pad39) -> COL0
- U1 pad 40: Net-(U1-Pad40) -> COL1
- U1 pad 41: Net-(U1-Pad41) -> COL2
Routing:
- net COL0: track 0.00 -> 85.1 mm, vias 0 -> 1
- net GND: track 0.00 -> 79.7 mm
- net +5V: track 0.00 -> 74.1 mm, vias 0 -> 4
- net ROW0: track 0.00 -> 67.0 mm
- net ROW1: track 0.00 -> 67.0 mm
- net COL1: track 0.00 -> 64.1 mm, vias 0 -> 1
- net COL3: track 0.00 -> 62.4 mm, vias 0 -> 1
- net COL2: track 0.00 -> 58.6 mm, vias 0 -> 1
- net Net-(D6-Pad2): track 0.00 -> 36.7 mm
- net Net-(D4-Pad2): track 0.00 -> 29.6 mm
- net Net-(D2-Pad2): track 0.00 -> 26.8 mm
- net VCC: track 0.00 -> 18.0 mm, vias 0 -> 1
- net Net-(J1-PadA5): track 0.00 -> 13.9 mm
- net Net-(D3-Pad2): track 0.00 -> 12.2 mm
- net Net-(D1-Pad2): track 0.00 -> 9.06 mm
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Other:
- net class Default: trace_width 0.25 -> 0.254
- net class Power added: clearance 0.2, trace_width 0.381, via_dia 0.8, via_drill 0.4
